File: Bus_switch.kicad_sch (KiCad schematic)
At the start: 8 parts, among them J3 Conn_01x04_Pin, U1 SN74CB3Q3384APW

Commit message: finished schematic
Parts:
- removed D1: LED, LED_SMD:LED_0603_1608Metric, symbol Device:LED
- removed J3: Conn_01x04_Pin, Connector_PinHeader_2.54mm:PinHeader_1x04_P2.54mm_Vertical, symbol Connector:Conn_01x04_Pin
- added D6: Red, PCM_JLCPCB:D_0603, symbol PCM_JLCPCB-Diodes:LED,0603,Red
- added R16, R17, R18, R2, R20, R22, R3: 10kΩ, PCM_JLCPCB:R_0402, symbol PCM_JLCPCB-Resistors:0402,10kΩ
- R4: now not fitted; now left out of the parts list
- renumbered R2 to R15, R3 to R19, R1 to R21
Connections:
- net +3V3: now also D6.2, R16.1, R17.1, R2.1, R22.2, R3.1; no longer R4.2
- net Chainbus.CS: now also R2.2
- net Chainbus.MISO: now also R18.1
- net Chainbus.MOSI: now also R20.1
- net Chainbus.RX: now also R17.2
- net Chainbus.SCK: now also R4.1, R3.2
- net Chainbus.TX: now also R16.2
- net GND: now also R4.2, R18.2, R20.2
- net SEL1: now also R22.1; no longer R4.1
- net at R21.2: now also D6.1
Other:
- note added: "Bus Pullups"
- note added: "You already have one, dude"
- note removed: "I2C Bus Pullup"
- note removed: "I2C pullup after bus switch"
- company: (none) -> Mini Moducard System
- moved on the sheet: C1, R15, R19, R21
