File: Interboard_connector.kicad_sch (KiCad schematic)
At the start: 2 parts, among them J1 Chainbus in, J2 Chainbus Out

Commit message: some schematic done
Other:
- title: MMS3 Stepper Controler -> MMS3 Hat template small (Change Me)
Changed lines of the file:
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@@
 	(paper "A4")
 	(title_block
-		(title "MMS3 Stepper Controler")
+		(title "MMS3 Hat template small (Change Me)")
 		(date "2026-02-25")
-		(rev "R0")
+		(rev "A")
 		(company "Moducard System")
 		(comment 1 "Made by Wojciech Szafrański")
