File: Interboard_connector.kicad_sch (KiCad schematic)
At the start: 2 parts, among them J1 Chainbus in, J2 Chainbus Out

Commit message: finished schematic
Other:
- company: Moducard System -> Mini Moducard System
