File: MMS3_hat_templates.kicad_sch (KiCad schematic)
At the start: 10 parts

Commit message: some schematic done
Parts:
- added C3, C5: 100nF, PCM_JLCPCB:C_0603, symbol PCM_JLCPCB-Capacitors:0603,100nF
- added C9: 100n, PCM_JLCPCB:C_0603, symbol Device:C
- added C? (x2): 10uF, PCM_JLCPCB:C_0603, symbol PCM_JLCPCB-Capacitors:0603,10uF
- added J4, J5: I2C_3V3, Connector_JST:JST_XH_S5B-XH-A_1x05_P2.50mm_Horizontal, symbol Connector:Conn_01x05_Pin
- added J6: Conn_01x03_Pin, Connector_PinSocket_2.54mm:PinSocket_1x03_P2.54mm_Vertical, symbol Connector:Conn_01x03_Pin
- added R10, R11, R12, R6, R7, R8, R9: 10kΩ, PCM_JLCPCB:R_0402, symbol PCM_JLCPCB-Resistors:0402,10kΩ
- added R5: 200kΩ, PCM_JLCPCB:R_0402, symbol PCM_JLCPCB-Resistors:0402,200kΩ
- added U3: PCA9306, symbol Interface:PCA9306
- added U6: TCA9535PWR, Package_SO:TSSOP-24_4.4x7.8mm_P0.65mm, symbol Interface_Expansion:TCA9535PWR
- added U?: AMS1117, PCM_JLCPCB:SOT-223-3_L6.5-W3.4-P2.30-LS7.0-BR, symbol PCM_JLCPCB-Power:LDO, 3.3V, 1A
Connections:
- net GND: now also C3.2, C5.2, C9.2, C?.2, C?.2, J4.1 (Pin_1), J5.1 (Pin_1), R11.1, R12.1, R8.1, U3.1 (GND), U6.12 (GND), U6.2 (A1), U6.21 (A0), U6.3 (A2), U?.1 (GND)
- new net: J4.3 (Pin_3), R7.2, U3.5 (SDA2)
- new net: J4.4 (Pin_4), R6.2, U3.6 (SCL2)
- new net: J6.2 (Pin_2), R5.1, R6.1, R7.1, U3.7 (VREF2)
- new net: R5.2, U3.8 (EN)
- new net +3V3: C5.1, C9.1, C?.1, J4.2 (Pin_2), J5.2 (Pin_2), J6.1 (Pin_1), R10.2, R9.2, U3.2 (VREF1), U6.24 (VCC), U?.2 (VOUT), U?.4 (VOUT)
- new net +5V: C3.1, C?.1, J4.5 (Pin_5), J5.5 (Pin_5), J6.3 (Pin_3), U?.3 (VIN)
- new net Chainbus.SCL: J5.4 (Pin_4), U3.3 (SCL1), U6.22 (SCL)
- new net Chainbus.SDA: J5.3 (Pin_3), U3.4 (SDA1), U6.23 (SDA)
- new net P00: R9.1, U6.4 (P00)
- new net P01: U6.5 (P01)
- new net P02: U6.6 (P02)
- new net P03: R8.2, U6.7 (P03)
- new net P04: U6.8 (P04)
- new net P05: U6.9 (P05)
- new net P06: U6.10 (P06)
- new net P07: R10.1, U6.11 (P07)
- new net P10: U6.13 (P10)
- new net P11: U6.14 (P11)
- new net P12: U6.15 (P12)
- new net P13: U6.16 (P13)
- new net P14: U6.17 (P14)
- new net P15: R11.2, U6.18 (P15)
- new net P16: U6.19 (P16)
- new net P17: U6.20 (P17)
- new net SPI 3/OE: R12.2
- no-connect marks 2 -> 1
Other:
- removed sheet Buck Regulator
- removed sheet Power Connector
- added sheet SPI 1 (SPI_Protocol_Connector.kicad_sch)
- added sheet SPI 2 (SPI_Protocol_Connector.kicad_sch)
- added sheet SPI 3 (SPI_Protocol_Connector.kicad_sch)
- added sheet UART 1 (UART_Protocol_Out.kicad_sch)
- added sheet UART 2 (UART_Protocol_Out.kicad_sch)
- note added: "3V3 LDO"
- note added: "GPIO expander"
- note added: "I2C"
- note added: "SPI 1"
- note added: "UART 1"
- note added: "UART 2"
- moved on the sheet: H1, H2, H3, H4, H5, H6, H7, H8, H9, PN1
