File: MMS3_hat_protocol.kicad_pcb (KiCad board)
At the start: 2 copper layers, 100 x 50 mm, 57 parts, among them J1 Chainbus in, J10 Conn_01x03_Pin, J11 Conn_01x04_Pin, J15 Conn_01x06_Pin, J2 Chainbus Out, J3 Conn_01x04_Pin, J4 Conn_01x04_Pin, J6 Conn_01x04_Pin, J7 Conn_01x04_Pin, J8 Conn_01x03_Pin, J9 Conn_01x03_Pin, U1 SN74CB3Q3384APW, U13 PCA9306, U2 M24C64, U3 AMS1117, U4 TXB0104PW, U5 TXB0104PW, U6 TCA9535PWR, U7 TXB0104PW, U8 TXB0104PW

Commit message: finished schematic
Parts:
- removed C12: 100nF, PCM_JLCPCB:C_0603
- removed C23: 100n, PCM_JLCPCB:C_0603
- removed D1: LED, LED_SMD:LED_0603_1608Metric
- removed J10: Conn_01x03_Pin, Connector_PinSocket_2.54mm:PinSocket_1x03_P2.54mm_Vertical
- removed J3: Conn_01x04_Pin, Connector_PinHeader_2.54mm:PinHeader_1x04_P2.54mm_Vertical
- removed R1: 330Ω, PCM_JLCPCB:R_0402
- removed U13: PCA9306, Package_SO:VSSOP-8_2.3x2mm_P0.5mm
- removed U6: TCA9535PWR, Package_SO:TSSOP-24_4.4x7.8mm_P0.65mm
- added C15: 100nF, PCM_JLCPCB:C_0603, F.Cu at (236.7, 117.7)
- added C17: 100nF, PCM_JLCPCB:C_0603, F.Cu at (236.7, 119.9)
- added C18: 100nF, PCM_JLCPCB:C_0603, F.Cu at (238.9, 98.9)
- added C19: 100nF, PCM_JLCPCB:C_0603, F.Cu at (238.9, 101.1)
- added C20: 100nF, PCM_JLCPCB:C_0603, F.Cu at (238.9, 103.4)
- added C21: 100nF, PCM_JLCPCB:C_0603, F.Cu at (238.9, 105.6)
- added D10: Red, PCM_JLCPCB:D_0603, F.Cu at (213.6, 94.3)
- added D6: Red, PCM_JLCPCB:D_0603, F.Cu at (219.6, 94.0)
- added D7: Red, PCM_JLCPCB:D_0603, F.Cu at (213.6, 86.5)
- added D8: Red, PCM_JLCPCB:D_0603, F.Cu at (213.6, 89.1)
- added D9: Red, PCM_JLCPCB:D_0603, F.Cu at (213.6, 91.7)
- added J12: Conn_01x04_Pin, Connector_JST:JST_XH_S4B-XH-A_1x04_P2.50mm_Horizontal, F.Cu at (121.2, 112.6)
- added J13: Conn_01x04_Pin, Connector_JST:JST_XH_S4B-XH-A_1x04_P2.50mm_Horizontal, F.Cu at (138.5, 113.0)
- added J14: Conn_01x03_Pin, Connector_PinSocket_2.54mm:PinSocket_1x03_P2.54mm_Vertical, F.Cu at (175.0, 113.0)
- added J5: Conn_01x03_Pin, Connector_PinSocket_2.54mm:PinSocket_1x03_P2.54mm_Vertical, F.Cu at (175.0, 122.0)
- added R10: 10kΩ, PCM_JLCPCB:R_0402, F.Cu at (218.9, 99.7)
- added R13: 330Ω, PCM_JLCPCB:R_0402, F.Cu at (218.9, 105.3)
- added R14: 330Ω, PCM_JLCPCB:R_0402, F.Cu at (218.9, 107.1)
- added R15: 10kΩ, PCM_JLCPCB:R_0402, F.Cu at (226.8, 116.7)
- added R16: 10kΩ, PCM_JLCPCB:R_0402, F.Cu at (226.8, 118.5)
- added R17: 10kΩ, PCM_JLCPCB:R_0402, F.Cu at (226.8, 120.4)
- added R18: 10kΩ, PCM_JLCPCB:R_0402, F.Cu at (226.8, 122.2)
- added R19: 10kΩ, PCM_JLCPCB:R_0402, F.Cu at (226.8, 124.1)
- added R20: 10kΩ, PCM_JLCPCB:R_0402, F.Cu at (226.8, 125.9)
- added R21: 330Ω, PCM_JLCPCB:R_0402, F.Cu at (226.8, 127.8)
- added R22: 10kΩ, PCM_JLCPCB:R_0402, F.Cu at (223.1, 93.6)
- added R6: 10kΩ, PCM_JLCPCB:R_0402, F.Cu at (216.1, 101.6)
- added U10: TXU0104PWR, TXU0104PWR:TSSOP-14_L5.0-W4.4-P0.65-LS6.4-BL, F.Cu at (138.0, 126.0)
- added U11: TXU0104PWR, TXU0104PWR:TSSOP-14_L5.0-W4.4-P0.65-LS6.4-BL, F.Cu at (128.0, 126.0)
- added U12: TXU0104PWR, TXU0104PWR:TSSOP-14_L5.0-W4.4-P0.65-LS6.4-BL, F.Cu at (146.0, 126.0)
- added U9: PCA9306DCUR, PCA9306DCUR:SSOP-8_L2.0-W2.3-P0.50-LS3.1-BR, F.Cu at (103.8, 123.4)
- J15: value Conn_01x06_Pin -> Conn_01x04_Pin; footprint Connector_JST:JST_XH_S6B-XH-A_1x06_P2.50mm_Horizontal -> Connector_JST:JST_XH_S4B-XH-A_1x04_P2.50mm_Horizontal
- J7: value Conn_01x04_Pin -> Conn_01x06_Pin; footprint Connector_JST:JST_XH_S4B-XH-A_1x04_P2.50mm_Horizontal -> Connector_JST:JST_XH_S6B-XH-A_1x06_P2.50mm_Horizontal
- J9: value Conn_01x03_Pin -> Conn_01x04_Pin; footprint Connector_PinSocket_2.54mm:PinSocket_1x03_P2.54mm_Vertical -> Connector_JST:JST_XH_S4B-XH-A_1x04_P2.50mm_Horizontal
- R12, R5: value 10kΩ -> 330Ω
- U4, U5, U8: value TXB0104PW -> TXU0104PWR; footprint Package_SO:TSSOP-14_4.4x5mm_P0.65mm -> TXU0104PWR:TSSOP-14_L5.0-W4.4-P0.65-LS6.4-BL
- U7: value TXB0104PW -> MAX3483ESA+T; footprint Package_SO:TSSOP-14_4.4x5mm_P0.65mm -> MAX3483ESA:PG-DSO-8_L5.0-W4.0-P1.27-LS6.0-BL
- moved C3 126.3 mm to (102.0, 100.0)
- moved C5 126.3 mm to (102.0, 102.2)
- moved R7 118.6 mm to (117.6, 131.6)
- moved R8 118.6 mm to (117.6, 133.5)
- moved R9 118.6 mm to (117.6, 135.3)
- moved U3 110.7 mm to (96.0, 102.0)
- moved U8 110.0 mm to (121.7, 126.0)
- moved U5 87.3 mm to (166.0, 126.0), turned to 90 degrees
- moved C2 84.0 mm to (242.9, 124.2), turned to 0 degrees
- moved C1 83.3 mm to (230.1, 125.4), turned to 0 degrees
- moved U1 79.7 mm to (222.3, 88.0), turned to 0 degrees
- moved R4 74.2 mm to (226.8, 114.8)
- moved R3 70.8 mm to (226.8, 113.0), turned to 0 degrees
- moved R2 63.9 mm to (219.0, 110.5)
- moved C7 52.1 mm to (217.3, 123.7)
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Connections:
- net Net-(J7-Pin_3) renamed /SPI 1/SCK_SEL
- net Net-(J7-Pin_4) renamed /SPI 1/MOSI_SEL
- C10 pad 1: +3V3 -> /SPI 1/V_SEL
- C11 pad 1: /SPI 1/V_2nd -> +3V3
- C13 pad 1: /SPI 1/V_2nd -> /UART 1/V_SEL
- C6 pad 1: GND -> +3V3
- C6 pad 2: /UART 1/V_2nd -> GND
- C7 pad 1: +3V3 -> /SPI 1/V_SEL
- C8 pad 1: GND -> +3V3
- C8 pad 2: /UART 2/V_2nd -> GND
- J11 pad 2: /UART 1/V_2nd -> /UART 1/V_SEL
- J11 pad 3: Net-(J11-Pin_3) -> /UART 1/RX_SEL
- J11 pad 4: Net-(J11-Pin_4) -> /UART 1/TX_SEL
- J15 pad 2: /SPI 1/V_2nd -> /UART 2/V_SEL
- J15 pad 3: Net-(J15-Pin_3) -> /UART 2/RX_SEL
- J15 pad 4: Net-(J15-Pin_4) -> /UART 2/TX_SEL
- J7 pad 2: /UART 2/V_2nd -> /SPI 1/V_SEL
- J9 pad 1: +3V3 -> /SPI 1/Bonus_IN_3_SEL
- J9 pad 2: /SPI 1/V_2nd -> /SPI 1/Bonus_IN_2_SEL
- J9 pad 3: +5V -> /SPI 1/Bonus_IN_1_SEL
- R12 pad 1: GND -> /P00
- R12 pad 2: /P03 -> Net-(D8-Pad2)
- R2 pad 2: /Chainbus.SCL -> /Chainbus.CS
- R3 pad 2: /Chainbus.SDA -> /Chainbus.SCK
- R4 pad 1: /Bus_switch/SEL1 -> /Chainbus.SCK
- R4 pad 2: +3V3 -> GND
- R5 pad 1: /P07 -> /P05
- R5 pad 2: +3V3 -> Net-(D7-Pad2)
- U4 pad 10: Net-(J17-Pin_2) -> /SPI 1/Bonus_OUT_1_SEL
- U4 pad 11: Net-(J17-Pin_3) -> /SPI 1/CS_SEL
- U4 pad 14: /UART 2/V_2nd -> /SPI 1/V_SEL
- U4 pad 2: /Chainbus.RX -> /Chainbus.MOSI
- U4 pad 3: /Chainbus.TX -> /Chainbus.SCK
- U4 pad 4: /P04 -> /Chainbus.CS
- U4 pad 5: /P05 -> /P17
- U4 pad 8: /P03 -> /P13
- U5 pad 1: +3V3 -> /SPI 1/V_SEL
- U5 pad 10: Net-(J18-Pin_2) -> /P14
- U5 pad 11: Net-(J18-Pin_3) -> /P15
- U5 pad 12: Net-(J11-Pin_3) -> /P16
- U5 pad 13: Net-(J11-Pin_4) -> /Chainbus.MISO
- U5 pad 14: /UART 1/V_2nd -> +3V3
- U5 pad 2: /Chainbus.RX -> /SPI 1/MISO_SEL
- U5 pad 3: /Chainbus.TX -> /SPI 1/Bonus_IN_1_SEL
- U5 pad 4: /P01 -> /SPI 1/Bonus_IN_2_SEL
- U5 pad 5: /P02 -> /SPI 1/Bonus_IN_3_SEL
- U5 pad 8: /P00 -> /P13
- U7 pad 1: +3V3 -> unconnected-(U7-RO-Pad1)
- U7 pad 2: /Chainbus.MISO -> unconnected-(U7-~{RE}-Pad2)
- U7 pad 3: /Chainbus.MOSI -> unconnected-(U7-DE-Pad3)
- U7 pad 4: /Chainbus.SCK -> unconnected-(U7-DI-Pad4)
- U7 pad 5: /P06 -> unconnected-(U7-GND-Pad5)
- U7 pad 7: GND -> unconnected-(U7-B-Pad7)
- U7 pad 8: /P07 -> unconnected-(U7-VCC-Pad8)
- U8 pad 1: +3V3 -> /UART 1/V_SEL
- U8 pad 10: unconnected-(U8-B4-Pad10) -> /UART 1/Bonus_IN_3_3V3
- U8 pad 11: unconnected-(U8-B3-Pad11) -> /UART 1/Bonus_IN_2_3V3
- U8 pad 12: unconnected-(U8-B2-Pad12) -> /P01
- U8 pad 13: unconnected-(U8-B1-Pad13) -> /Chainbus.RX
- U8 pad 14: /SPI 1/V_2nd -> +3V3
- U8 pad 2: /P10 -> /UART 1/RX_SEL
- U8 pad 3: /P11 -> /UART 1/Bonus_IN_1_SEL
- U8 pad 4: /P12 -> /UART 1/Bonus_IN_2_SEL
- U8 pad 5: /P13 -> /UART 1/Bonus_IN_3_SEL
- U8 pad 8: /P07 -> /P00
Routing:
- net /Bus_switch/SEL1: track 83.6 -> 20.6 mm, vias 2 -> 0
- net /Chainbus.SCL: track 31.8 -> 0.00 mm, vias 2 -> 0
- net /Chainbus.SDA: track 30.3 -> 0.00 mm, vias 1 -> 0
- net +3V3: track 27.3 -> 0.00 mm, vias 1 -> 0
- net /Bus_switch/Chainbus_In.SDA: track 20.4 -> 2.04 mm, vias 2 -> 1
- net /Bus_switch/Chainbus_In.SCL: track 18.5 -> 2.09 mm, vias 2 -> 1
- net /Bus_switch/Chainbus_In.CS: track 14.2 -> 2.11 mm
- net /Bus_switch/Chainbus_In.MOSI: track 7.70 -> 2.02 mm
- net /Bus_switch/Chainbus_In.SCK: track 7.52 -> 1.93 mm
- net /Bus_switch/Chainbus_In.MISO: track 6.11 -> 2.02 mm
- net /Bus_switch/Chainbus_In.TX: track 6.24 -> 2.39 mm
- net /Bus_switch/Chainbus_In.RX: track 5.76 -> 2.31 mm
- net Net-(D1-A): track 1.52 -> 0.00 mm
- net (no net): track 0.00 -> 1.52 mm
Other:
- outline, holes or cut-outs redrawn
- board text added: "Front and Back keepout zone for DIN rail mount"
- board text added: "Version 1.0 Made by Wojciech Szafrański"
- board text removed: "GND"
