File: SPI_Protocol_Connector.kicad_sch (KiCad schematic)
At the start: 8 parts, among them J5 Conn_01x03_Pin, J7 Conn_01x06_Pin, U4 TXU0104PWR, U5 TXU0104PWR

Commit message: finished schematic
Parts:
- J5: footprint Connector_PinSocket_2.54mm:PinSocket_1x03_P2.54mm_Vertical -> Connector_PinSocket_2.54mm:PinSocket_1x03_P2.54mm_Horizontal
Other:
- company: (none) -> Mini Moducard System
