File: UART_Protocol_Connector.kicad_sch (KiCad schematic)
At the start: 8 parts, among them J11 Conn_01x04_Pin, J8 Conn_01x03_Pin, U11 TXU0104PWR, U8 TXU0104PWR

Commit message: finished schematic
Parts:
- added C12: 100nF, PCM_JLCPCB:C_0603, symbol PCM_JLCPCB-Capacitors:0603,100nF
- added D11, D13: Red, PCM_JLCPCB:D_0603, symbol PCM_JLCPCB-Diodes:LED,0603,Red
- added R23, R26: 510Ω, PCM_JLCPCB:R_0603, symbol PCM_JLCPCB-Resistors:0603,510Ω
- added R25: 120Ω, PCM_JLCPCB:R_0603, symbol PCM_JLCPCB-Resistors:0603,120Ω
- added R29, R31: 330Ω, PCM_JLCPCB:R_0402, symbol PCM_JLCPCB-Resistors:0402,330Ω
- added R33, R35: 10kΩ, PCM_JLCPCB:R_0402, symbol PCM_JLCPCB-Resistors:0402,10kΩ
- added U6: MAX13487EESA, MAX13487EESA:SOIC-8_L4.9-W3.9-P1.27-LS6.0-BL, symbol MAX13487EESA:MAX13487EESA
- J8: footprint Connector_PinSocket_2.54mm:PinSocket_1x03_P2.54mm_Vertical -> Connector_PinSocket_2.54mm:PinSocket_1x03_P2.54mm_Horizontal
Connections:
- net +3V3: now also D11.2, D13.2, R33.2, R35.1
- net +5V: now also C12.1, R23.2, U6.8 (VCC)
- net Chainbus.RX: now also U6.1 (RO)
- net Chainbus.TX: now also U6.4 (DI)
- net GND: now also C12.2, R26.1, U6.5 (GND)
- net Bonus_IN_3_3V3: no longer names the net of U8.10 (B4Y)
- net Bonus_IN_3_SEL: no longer names the net of U8.5 (A4)
- net Bonus_OUT_3_3V3: no longer names the net of U11.5 (A4)
- net Bonus_OUT_3_SEL: no longer names the net of U11.10 (B4Y)
- net OE renamed UART_OE
- net RX_SEL renamed RS485_A
- net RS485_A: now also R23.1, R25.2, U6.6 (A)
- net TX_SEL renamed RS485_B
- net RS485_B: now also R25.1, R26.2, U6.7 (B)
- new net: D11.1, R29.2
- new net: D13.1, R31.2
- new net RS485_Reciever_enable_NEGATED: R31.1, R33.1, U6.2 (~{RE})
- new net RS485_Shutdown_NEGATED: R29.1, R35.2, U6.3 (~{SHDN})
- no-connect marks 4 -> 8
Other:
- note added: "Default: MAX13487EESA - 0.25Mbps, better emi resistance Drop in replacement: MAX13488EESA+- 12Mbps, worse emi resistance"
- note added: "RO = VCC-1.5V"
- note added: "RS485 Converter"
- note added: "Resistors are required for RS-485 R23 R26 are to pullup/down the bus to stable voltage in case of of open-circuit bus condition R25 is terminating resistor Shouldn't be soldered when using UART Should be soldered when using RS-485"
- note added: "UART and RS485"
- note removed: "UART"
- company: (none) -> Mini Moducard System
- moved on the sheet: C13, C15, C17, C6, J11, U11, U8
