File: Hardware/MMS3_hat_protocol.kicad_sch (KiCad schematic)
At the start: 64 parts, among them J10 Conn_01x02_Pin, J3 Conn_01x02_Pin, J4 Conn_01x04_Pin, J6 Conn_01x04_Pin, J9 Conn_01x04_Pin, U13 TCA9535PWR_C130204, U3 AMS1117, U9 PCA9306DCUR

Commit message: V1.1, added photo
Parts:
- removed H7, H8, H9: (no value), PCM_JLCPCB:Hole_Tooling_JLCPCB, symbol PCM_JLCPCB-Manufacturing:Tooling Hole, PCM_JLCPCB, 1.152mm
Connections:
- net +3V3: now also D15.2, D16.2, D17.2, D18.2; no longer D15.1, D16.1, D17.1, D18.1
- net at R37.2: now also D15.1; no longer D15.2
- net at R39.2: now also D16.1; no longer D16.2
- net at R43.2: now also D18.1; no longer D18.2
- net at R41.2: now also D17.1; no longer D17.2
Other:
- moved on the sheet: D15, D16, D17, D18
